Commit message: set gripper to mimic

File: src/piper_description/urdf/piper_description.xacro (robot description, xacro)
@@ -507,5 +507,5 @@
       link="link8" />
     <axis
-      xyz="0 0 1" />
+      xyz="0 0 -1" />
     <limit
       lower="-0.04"
@@ -513,4 +513,5 @@
       effort="10"
       velocity="1" />
+    <mimic joint="joint7"/>
   </joint>
 <!-- controller -->
